File: fpgafmctl.sch (EAGLE design)
At the start: 10 parts, among them IC1 ATTINY45-20P

Commit message: update schem
Parts:
- added S1: (no value), switch-omron:31-XX
Connections:
- new net N$1: IC1.(XTAL1/CLKI/OC1B/ADC3/PCINT3)PB3, S1.S
- net GND: now also S1.P
Changed lines of the file:
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@@
 <part name="SUPPLY1" library="supply2" deviceset="VCC" device=""/>
 <part name="JP2" library="sparkfun" deviceset="M20" device=""/>
+<part name="S1" library="switch-omron" deviceset="31-XX" device=""/>
 </parts>
 <sheets>
@@
 <instance part="SUPPLY1" gate="G$1" x="91.44" y="68.58"/>
 <instance part="JP2" gate="G$1" x="-30.48" y="40.64"/>
+<instance part="S1" gate="1" x="114.3" y="20.32"/>
 </instances>
 <busses>
@@
 <wire x1="129.54" y1="20.32" x2="129.54" y2="12.7" width="0.1524" layer="91"/>
 <pinref part="C2" gate="G$1" pin="-"/>
-<wire x1="99.06" y1="12.7" x2="129.54" y2="12.7" width="0.1524" layer="91"/>
+<wire x1="99.06" y1="12.7" x2="114.3" y2="12.7" width="0.1524" layer="91"/>
 <junction x="15.24" y="53.34"/>
 <junction x="99.06" y="12.7"/>
 <pinref part="R1" gate="G$1" pin="1"/>
+<wire x1="114.3" y1="12.7" x2="129.54" y2="12.7" width="0.1524" layer="91"/>
 <wire x1="17.78" y1="88.9" x2="15.24" y2="88.9" width="0.1524" layer="91"/>
 <wire x1="15.24" y1="88.9" x2="15.24" y2="63.5" width="0.1524" layer="91"/>
 <junction x="15.24" y="63.5"/>
+<pinref part="S1" gate="1" pin="P"/>
+<wire x1="114.3" y1="15.24" x2="114.3" y2="12.7" width="0.1524" layer="91"/>
+<junction x="114.3" y="12.7"/>
 </segment>
 </net>
@@
 </segment>
 </net>
+<net name="N$1" class="0">
+<segment>
+<pinref part="IC1" gate="G$1" pin="(XTAL1/CLKI/OC1B/ADC3/PCINT3)PB3"/>
+<wire x1="99.06" y1="48.26" x2="114.3" y2="48.26" width="0.1524" layer="91"/>
+<pinref part="S1" gate="1" pin="S"/>
+<wire x1="114.3" y1="48.26" x2="114.3" y2="25.4" width="0.1524" layer="91"/>
+</segment>
+</net>
